File: mcu.kicad_sch (KiCad schematic)
At the start: 35 parts, among them J1 Conn_ST_STDC14, SW1 RESET, Y1 16MHz

Commit message: fix: chip selects
Connections:
- net LED_1: now also IC?.82 (PD13)
- net LED_2: now also IC?.81 (PD12)
- net SPI2_CSS: now reaches IC?.29 (PC3_C)
- net SPI3_CSS: now reaches IC?.47 (PB1)
- net SPI1_NSS renamed SPI1_CSS
- net SPI2_NSS: no longer names the net of IC?.140 (PB9)
- net SPI3_NSS: no longer names the net of IC?.40 (PA4)
Changed lines of the file:
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@@
 	(wire
 		(pts
-			(xy 175.26 74.93) (xy 175.26 80.01)
+			(xy 153.67 168.91) (xy 157.48 168.91)
 		)
 		(stroke
@@
 	(wire
 		(pts
+			(xy 261.62 163.83) (xy 273.05 163.83)
+		)
+		(stroke
+			(width 0)
+			(type default)
+		)
+	)
+	(wire
+		(pts
 			(xy 38.1 134.62) (xy 38.1 154.94)
 		)
@@
 	(wire
 		(pts
-			(xy 172.72 204.47) (xy 172.72 209.55)
+			(xy 190.5 204.47) (xy 190.5 209.55)
 		)
 		(stroke
@@
 	(wire
 		(pts
+			(xy 261.62 166.37) (xy 273.05 166.37)
+		)
+		(stroke
+			(width 0)
+			(type default)
+		)
+	)
+	(wire
+		(pts
 			(xy 261.62 179.07) (xy 273.05 179.07)
 		)
@@
 		)
 	)
+	(label "LED_1"
+		(at 273.05 163.83 180)
+		(effects
+			(font
+				(size 1.27 1.27)
+			)
+			(justify right bottom)
+		)
+	)
 	(label "VDD_8"
 		(at 273.05 97.79 180)
@@
 		)
 	)
+	(label "LED_2"
+		(at 273.05 166.37 180)
+		(effects
+			(font
+				(size 1.27 1.27)
+			)
+			(justify right bottom)
+		)
+	)
 	(label "OSC_OUT"
 		(at 146.05 156.21 0)
@@
 		)
 	)
-	(hierarchical_label "SPI2_NSS"
+	(hierarchical_label "SPI2_CSS"
 		(shape output)
-		(at 175.26 74.93 90)
+		(at 153.67 168.91 180)
 		(effects
 			(font
 				(size 1.27 1.27)
 			)
-			(justify left)
+			(justify right)
 		)
 	)
@@
 		)
 	)
-	(hierarchical_label "SPI1_NSS"
+	(hierarchical_label "SPI1_CSS"
 		(shape output)
 		(at 213.36 76.2 90)
@@
 		)
 	)
-	(hierarchical_label "SPI3_NSS"
-		(shape input)
-		(at 172.72 209.55 270)
+	(hierarchical_label "SPI3_CSS"
+		(shape output)
+		(at 190.5 209.55 270)
 		(effects
 			(font

Commit message: feat: setup micro on pcb
Parts:
- gave numbers to parts that had none: 1
Changed lines of the file:
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@@
 		(dnp no)
 		(fields_autoplaced yes)
-		(property "Reference" "IC?"
+		(property "Reference" "IC5"
 			(at 265.43 91.4714 0)
 			(effects
@@
 			(project "axes-controller-board"
 				(path "/88591975-6c45-4e1d-8f38-0b5760acfc98/37bdac2b-aaa0-48b9-94b0-0180a23198dc"
-					(reference "IC?")
+					(reference "IC5")
 					(unit 1)
 				)

Commit message: feat: setup groups pcb
steppers, micro, clock, current sensor - connector
Connections:
- net GND: now also IC5.94 (VSS_6)
Changed lines of the file:
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@@
 	)
 	(junction
+		(at 54.61 78.74)
+		(diameter 0)
+		(color 0 0 0 0)
+	)
+	(junction
 		(at 54.61 67.31)
 		(diameter 0)
@@
 	(wire
 		(pts
+			(xy 261.62 133.35) (xy 274.32 133.35)
+		)
+		(stroke
+			(width 0)
+			(type default)
+		)
+	)
+	(wire
+		(pts
 			(xy 203.2 204.47) (xy 203.2 214.63)
 		)
@@
 	(wire
 		(pts
+			(xy 54.61 78.74) (xy 63.5 78.74)
+		)
+		(stroke
+			(width 0)
+			(type default)
+		)
+	)
+	(wire
+		(pts
 			(xy 151.13 181.61) (xy 157.48 181.61)
 		)
@@
 		)
 	)
+	(label "VSS_6"
+		(at 63.5 78.74 180)
+		(effects
+			(font
+				(size 1.27 1.27)
+			)
+			(justify right bottom)
+		)
+	)
 	(label "VDD_6"
 		(at 254 214.63 90)
@@
 		(effects
 			(font
+				(size 1.27 1.27)
+			)
+			(justify right bottom)
+		)
+	)
+	(label "VSS_6"
+		(at 274.32 133.35 180)
+		(effects
+			(font

Commit message: feat: endstops integration
Connections:
- net ES_Y2: now reaches IC5.90 (PG5)
- net ES_Y1: now reaches IC5.91 (PG6)
- net ES_X: now reaches IC5.92 (PG7)
Changed lines of the file:
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@@
+	(wire
+		(pts
+			(xy 261.62 140.97) (xy 266.7 140.97)
+		)
+		(stroke
+			(width 0)
+			(type default)
+		)
+	)
 	(wire
 		(pts
@@
 	(wire
 		(pts
+			(xy 261.62 143.51) (xy 266.7 143.51)
+		)
+		(stroke
+			(width 0)
+			(type default)
+		)
+	)
+	(wire
+		(pts
 			(xy 190.5 204.47) (xy 190.5 209.55)
 		)
@@
 		(pts
 			(xy 67.31 199.39) (xy 67.31 198.12)
+		)
+		(stroke
+			(width 0)
+			(type default)
+		)
+	)
+	(wire
+		(pts
+			(xy 261.62 138.43) (xy 266.7 138.43)
 		)
 		(stroke
@@
 		)
 	)
+	(hierarchical_label "ES_X"
+		(shape input)
+		(at 266.7 138.43 0)
+		(effects
+			(font
+				(size 1.27 1.27)
+			)
+			(justify left)
+		)
+	)
 	(hierarchical_label "X_DC_PWM_1"
 		(shape output)
@@
 		)
 	)
+	(hierarchical_label "ES_Y1"
+		(shape input)
+		(at 266.7 140.97 0)
+		(effects
+			(font
+				(size 1.27 1.27)
+			)
+			(justify left)
+		)
+	)
 	(hierarchical_label "Y1_DC_PWM_1"
 		(shape output)
@@
 		(effects
 			(font
+				(size 1.27 1.27)
+			)
+			(justify left)
+		)
+	)
+	(hierarchical_label "ES_Y2"
+		(shape input)
+		(at 266.7 143.51 0)
+		(effects
+			(font

Commit message: feat: spi and 3v3 routing
Parts:
- added R19, R20, R21, R22, R23, R24, R25, R26, R27, R28, R29, R30, R31, R32, R4, R5, R6, R7: R, Resistor_SMD:R_0603_1608Metric, symbol Device:R
Connections:
- net DIR_F: now also R6.2; no longer IC5.58 (PE7)
- net DIR_P1: now also R25.1; no longer IC5.115 (PD1)
- net DIR_P2: now also R24.1; no longer IC5.118 (PD4)
- net DIR_Y: now also R5.2; no longer IC5.79 (PD10)
- net DIR_Z1: now also R22.1; no longer IC5.142 (PE1)
- net DIR_Z2: now also R20.1; no longer IC5.3 (PE4)
- net STEP_F: now also R7.1; no longer IC5.59 (PE8)
- net STEP_P1: now also R26.2; no longer IC5.114 (PD0)
- net STEP_P2: now also R23.2; no longer IC5.117 (PD3)
- net STEP_Y: now also R4.2; no longer IC5.80 (PD11)
- net STEP_Z1: now also R21.2; no longer IC5.141 (PE0)
- net STEP_Z2: now also R19.2; no longer IC5.2 (PE3)
- net X_DC_PWM_1: now also R32.2; no longer IC5.60 (PE9)
- net X_DC_PWM_2: now also R31.1; no longer IC5.64 (PE11)
- net Y1_DC_PWM_1: now also R29.1; no longer IC5.66 (PE13)
- net Y1_DC_PWM_2: now also R30.1; no longer IC5.67 (PE14)
- net Y2_DC_PWM_1: now also R28.2; no longer IC5.96 (PC6)
- net Y2_DC_PWM_2: now also R27.2; no longer IC5.97 (PC7)
- new net: IC5.118 (PD4), R24.2
- new net: IC5.64 (PE11), R31.2
- new net: IC5.115 (PD1), R25.2
- new net: IC5.114 (PD0), R26.1
- new net: IC5.141 (PE0), R21.1
- new net: IC5.3 (PE4), R20.2
- new net: IC5.2 (PE3), R19.1
- new net: IC5.79 (PD10), R5.1
- new net: IC5.97 (PC7), R27.1
- new net: IC5.60 (PE9), R32.1
- new net: IC5.59 (PE8), R7.2
- new net: IC5.80 (PD11), R4.1
- new net: IC5.66 (PE13), R29.2
- new net: IC5.117 (PD3), R23.1
- new net: IC5.58 (PE7), R6.1
- new net: IC5.142 (PE1), R22.2
- new net: IC5.67 (PE14), R30.2
- new net: IC5.96 (PC6), R28.1

Commit message: fix: minors
Connections:
- net ES_Z1: now reaches IC5.88 (PG3)
- net ES_Z2: now reaches IC5.89 (PG4)
Changed lines of the file:
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@@
+	(wire
+		(pts
+			(xy 261.62 146.05) (xy 266.7 146.05)
+		)
+		(stroke
+			(width 0)
+			(type default)
+		)
+	)
 	(wire
 		(pts
@@
 		(pts
 			(xy 38.1 154.94) (xy 41.91 154.94)
+		)
+		(stroke
+			(width 0)
+			(type default)
+		)
+	)
+	(wire
+		(pts
+			(xy 261.62 148.59) (xy 266.7 148.59)
 		)
 		(stroke
@@
 		)
 	)
+	(hierarchical_label "ES_Z1"
+		(shape input)
+		(at 266.7 148.59 0)
+		(effects
+			(font
+				(size 1.27 1.27)
+			)
+			(justify left)
+		)
+	)
 	(hierarchical_label "STEP_P2"
 		(shape output)
@@
 		(effects
 			(font
+				(size 1.27 1.27)
+			)
+			(justify left)
+		)
+	)
+	(hierarchical_label "ES_Z2"
+		(shape input)
+		(at 266.7 146.05 0)
+		(effects
+			(font

Commit message: fix: ground planes
Parts:
- C4, C5: value C -> 15pF
- R3: value R -> 33R
Changed lines of the file:
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@@
 		(fields_autoplaced yes)
 		(property "Reference" "R3"
-			(at 33.02 193.04 90)
+			(at 33.02 191.77 90)
 			(effects
 				(font
@@
 			)
 		)
-		(property "Value" "R"
-			(at 33.02 195.58 90)
+		(property "Value" "33R"
+			(at 33.02 194.31 90)
 			(effects
 				(font
@@
 		(fields_autoplaced yes)
 		(property "Reference" "C4"
-			(at 46.99 201.93 0)
+			(at 46.99 201.9299 0)
 			(effects
 				(font
@@
 			)
 		)
-		(property "Value" "C"
-			(at 46.99 204.47 0)
+		(property "Value" "15pF"
+			(at 46.99 204.4699 0)
 			(effects
 				(font
@@
 		(fields_autoplaced yes)
 		(property "Reference" "C5"
-			(at 71.12 201.93 0)
+			(at 71.12 201.9299 0)
 			(effects
 				(font
@@
 			)
 		)
-		(property "Value" "C"
-			(at 71.12 204.47 0)
+		(property "Value" "15pF"
+			(at 71.12 204.4699 0)
 			(effects
 				(font

Commit message: feat: nozzle and hb connections
Parts:
- added R43, R44: R, Resistor_SMD:R_0603_1608Metric, symbol Device:R
Connections:
- net N_NTC: now reaches IC5.36 (PA2)
- net H_NTC: now reaches IC5.37 (PA3)
- net at IC5.85 (PD14): now also R44.2
- net at IC5.86 (PD15): now also R43.2
- new net H_PWM: R44.1
- new net N_PWM: R43.1
Changed lines of the file:
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@@
 	(wire
 		(pts
+			(xy 151.13 186.69) (xy 157.48 186.69)
+		)
+		(stroke
+			(width 0)
+			(type default)
+		)
+	)
+	(wire
+		(pts
 			(xy 152.4 115.57) (xy 157.48 115.57)
 		)
@@
 	(wire
 		(pts
+			(xy 275.59 153.67) (xy 261.62 153.67)
+		)
+		(stroke
+			(width 0)
+			(type default)
+		)
+	)
+	(wire
+		(pts
 			(xy 111.76 39.37) (xy 101.6 39.37)
 		)
@@
 	(wire
 		(pts
+			(xy 275.59 156.21) (xy 261.62 156.21)
+		)
+		(stroke
+			(width 0)
+			(type default)
+		)
+	)
+	(wire
+		(pts
 			(xy 248.92 76.2) (xy 248.92 80.01)
 		)
@@
 	(wire
 		(pts
+			(xy 165.1 204.47) (xy 165.1 215.9)
+		)
+		(stroke
+			(width 0)
+			(type default)
+		)
+	)
+	(wire
+		(pts
 			(xy 97.79 77.47) (xy 101.6 77.47)
 		)
@@
 		)
 	)
+	(hierarchical_label "N_NTC"
+		(shape input)
+		(at 151.13 186.69 180)
+		(effects
+			(font
+				(size 1.27 1.27)
+			)
+			(justify right)
+		)
+	)
 	(hierarchical_label "DIR_P2"
 		(shape output)
@@
 		)
 	)
+	(hierarchical_label "N_PWM"
+		(shape output)
+		(at 283.21 153.67 0)
+		(effects
+			(font
+				(size 1.27 1.27)
+			)
+			(justify left)
+		)
+	)
 	(hierarchical_label "X_DC_PWM_2"
 		(shape output)
@@
 		)
 	)
+	(hierarchical_label "H_PWM"
+		(shape output)
+		(at 283.21 156.21 0)
+		(effects
+			(font
+				(size 1.27 1.27)
+			)
+			(justify left)
+		)
+	)
 	(hierarchical_label "Y1_DC_PWM_2"
 		(shape output)
@@
 		)
 	)
+	(hierarchical_label "H_NTC"
+		(shape input)
+		(at 165.1 215.9 270)
+		(effects
+			(font
+				(size 1.27 1.27)
+			)
+			(justify right)
+		)
+	)
 	(hierarchical_label "MY1_A"
 		(shape input)
@@
 	(symbol
 		(lib_id "Device:R")
+		(at 279.4 153.67 270)
+		(unit 1)
+		(exclude_from_sim no)
+		(in_bom yes)
+		(on_board yes)
+		(dnp no)
+		(property "Reference" "R43"
+			(at 274.574 152.654 90)
+			(effects
+				(font
+					(size 1.27 1.27)
+				)
+			)
+		)
+		(property "Value" "R"
+			(at 279.4 153.67 90)
+			(effects
+				(font
+					(size 1.27 1.27)
+				)
+			)
+		)
+		(property "Footprint" "Resistor_SMD:R_0603_1608Metric"
+			(at 279.4 151.892 90)
+			(effects
+				(font
+					(size 1.27 1.27)
+				)
+				(hide yes)
+			)
+		)
+		(property "Datasheet" "~"
+			(at 279.4 153.67 0)
+			(effects
+				(font
+					(size 1.27 1.27)
+				)
+				(hide yes)
+			)
+		)
+		(property "Description" ""
+			(at 279.4 153.67 0)
+			(effects
+				(font
+					(size 1.27 1.27)
+				)
+				(hide yes)
+			)
+		)
+		(pin "1"
+		)
+		(pin "2"
+		)
+		(instances
+			(project "axes-controller-board"
+				(path "/88591975-6c45-4e1d-8f38-0b5760acfc98/37bdac2b-aaa0-48b9-94b0-0180a23198dc"
+					(reference "R43")
+					(unit 1)
+				)
+			)
+		)
+	)
+	(symbol
+		(lib_id "Device:R")
 		(at 278.13 168.91 90)
 		(unit 1)
@@
 					(unit 1)
 				)
+			)
+		)
+	)
+	(symbol
+		(lib_id "Device:R")
+		(at 279.4 156.21 270)
+		(unit 1)
+		(exclude_from_sim no)
+		(in_bom yes)
+		(on_board yes)
+		(dnp no)
+		(property "Reference" "R44"
+			(at 274.828 155.194 90)
+			(effects
+				(font
+					(size 1.27 1.27)
+				)
+			)
+		)
+		(property "Value" "R"
+			(at 279.4 156.21 90)
+			(effects
+				(font
+					(size 1.27 1.27)
+				)
+			)
+		)
+		(property "Footprint" "Resistor_SMD:R_0603_1608Metric"
+			(at 279.4 154.432 90)
+			(effects
+				(font
+					(size 1.27 1.27)
+				)
+				(hide yes)
+			)
+		)
+		(property "Datasheet" "~"
+			(at 279.4 156.21 0)
+			(effects
+				(font
+					(size 1.27 1.27)
+				)
+				(hide yes)
+			)
+		)
+		(property "Description" ""
+			(at 279.4 156.21 0)
+			(effects
+				(font
+					(size 1.27 1.27)
+				)
+				(hide yes)
+			)
+		)
+		(pin "1"
+		)
+		(pin "2"
+		)
+		(instances
+			(project "axes-controller-board"
+				(path "/88591975-6c45-4e1d-8f38-0b5760acfc98/37bdac2b-aaa0-48b9-94b0-0180a23198dc"
+					(reference "R44")
+					(unit 1)
+				)
