File: sensors.kicad_sch (KiCad schematic)
At the start: 42 parts, among them IC2 ACS37800KMACTR-030B3-SPI, IC3 ACS37800KMACTR-030B3-SPI, IC4 ACS37800KMACTR-030B3-SPI, U3 UA9637A, U5 UA9637A, U7 UA9637A

Commit message: chore: add CERN-OHL-S-2.0 license, README and fabrication outputs
Stop tracking third-party SamacSys/vendor models and datasheets, which
may not be redistributed as library parts.

Co-Authored-By: Claude Opus 5.5 <noreply@anthropic.com>
Other:
- company: (none) -> Leonardo Pasquato
Changed lines of the file:
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@@
 	(generator_version "8.0")
 	(paper "A3")
+	(title_block
+		(rev "1.0.0")
+		(company "Leonardo Pasquato")
+		(comment 1 "Copyright 2026 Leonardo Pasquato")
+		(comment 2 "Licensed under CERN-OHL-S-2.0, https://ohwr.org/cern_ohl_s_v2.txt")
+		(comment 3 "Source: https://github.com/DEDALUS-5x/axes-controller-board")
+		(comment 4 "Distributed WITHOUT ANY WARRANTY, see LICENSE")
+	)
 	(junction
 		(at 312.42 167.64)
